File: jumpers.kicad_sch (KiCad schematic)
At the start: 2 parts, among them J5 Conn_02x09_Odd_Even, J6 Conn_02x06_Odd_Even

Commit message: PCB layout done, signal routing finished, power routing remaining.
Parts:
- renumbered J6 to J5, J5 to J6
Changed lines of the file:
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@@
 		(dnp no)
 		(fields_autoplaced yes)
-		(property "Reference" "#PWR056"
+		(property "Reference" "#PWR058"
 			(at 137.16 111.76 0)
 			(hide yes)
@@
 			(project "DigiFur-Rev1.0"
 				(path "/54298b52-0ffe-40ef-8666-22993c0ca2db"
-					(reference "#PWR056")
+					(reference "#PWR058")
 					(unit 1)
 				)
@@
 		(dnp no)
 		(fields_autoplaced yes)
-		(property "Reference" "#PWR060"
+		(property "Reference" "#PWR057"
 			(at 137.16 55.88 0)
 			(hide yes)
@@
 			(project "DigiFur-Rev1.0"
 				(path "/54298b52-0ffe-40ef-8666-22993c0ca2db"
-					(reference "#PWR060")
+					(reference "#PWR057")
 					(unit 1)
 				)
@@
 		(dnp no)
 		(fields_autoplaced yes)
-		(property "Reference" "#PWR057"
+		(property "Reference" "#PWR060"
 			(at 139.7 142.24 0)
 			(hide yes)
@@
 			(project "DigiFur-Rev1.0"
 				(path "/54298b52-0ffe-40ef-8666-22993c0ca2db"
-					(reference "#PWR057")
+					(reference "#PWR060")
 					(unit 1)
 				)
@@
 		(in_pos_files yes)
 		(dnp no)
-		(property "Reference" "J5"
+		(property "Reference" "J6"
 			(at 148.59 106.68 0)
 			(show_name no)
@@
 			(project "DigiFur-Rev1.0"
 				(path "/54298b52-0ffe-40ef-8666-22993c0ca2db"
-					(reference "J5")
+					(reference "J6")
 					(unit 1)
 				)
@@
 		(dnp no)
 		(fields_autoplaced yes)
-		(property "Reference" "#PWR058"
+		(property "Reference" "#PWR062"
 			(at 157.48 142.24 0)
 			(hide yes)
@@
 			(project "DigiFur-Rev1.0"
 				(path "/54298b52-0ffe-40ef-8666-22993c0ca2db"
-					(reference "#PWR058")
+					(reference "#PWR062")
 					(unit 1)
 				)
@@
 		(in_pos_files yes)
 		(dnp no)
-		(property "Reference" "J6"
+		(property "Reference" "J5"
 			(at 148.59 52.07 0)
 			(show_name no)
@@
 			(project "DigiFur-Rev1.0"
 				(path "/54298b52-0ffe-40ef-8666-22993c0ca2db"
-					(reference "J6")
+					(reference "J5")
 					(unit 1)
 				)
@@
 		(dnp no)
 		(fields_autoplaced yes)
-		(property "Reference" "#PWR059"
+		(property "Reference" "#PWR064"
 			(at 160.02 111.76 0)
 			(hide yes)
@@
 			(project "DigiFur-Rev1.0"
 				(path "/54298b52-0ffe-40ef-8666-22993c0ca2db"
-					(reference "#PWR059")
+					(reference "#PWR064")
 					(unit 1)
 				)
@@
 		(dnp no)
 		(fields_autoplaced yes)
-		(property "Reference" "#PWR061"
+		(property "Reference" "#PWR059"
 			(at 139.7 76.2 0)
 			(hide yes)
@@
 			(project "DigiFur-Rev1.0"
 				(path "/54298b52-0ffe-40ef-8666-22993c0ca2db"
-					(reference "#PWR061")
+					(reference "#PWR059")
 					(unit 1)
 				)
@@
 		(dnp no)
 		(fields_autoplaced yes)
-		(property "Reference" "#PWR062"
+		(property "Reference" "#PWR061"
 			(at 157.48 76.2 0)
 			(hide yes)
@@
 			(project "DigiFur-Rev1.0"
 				(path "/54298b52-0ffe-40ef-8666-22993c0ca2db"
-					(reference "#PWR062")
-					(unit 1)
-				)
+					(reference "#PWR061")
+					(unit 1)
+				)

Commit message: Revision to fix problems from first board fab
Parts:
- added R63: 10k, Resistor_SMD:R_0603_1608Metric_Pad0.98x0.95mm_HandSolder, symbol Device:R_Small
Connections:
- net +3.3V_MCU: now also R63.1; no longer J5.8 (Pin_8)
- new net: J5.8 (Pin_8), R63.2
Changed lines of the file:
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@@
 	(paper "A4")
+	(junction
+		(at 157.48 46.99)
+		(diameter 0)
+		(color 0 0 0 0)
+	)
 	(junction
 		(at 139.7 130.81)
@@
 		(color 0 0 0 0)
 	)
-	(junction
-		(at 160.02 54.61)
-		(diameter 0)
-		(color 0 0 0 0)
-	)
 	(wire
 		(pts
@@
 	(wire
 		(pts
+			(xy 154.94 54.61) (xy 157.48 54.61)
+		)
+		(stroke
+			(width 0)
+			(type default)
+		)
+	)
+	(wire
+		(pts
 			(xy 157.48 115.57) (xy 157.48 130.81)
 		)
@@
 	(wire
 		(pts
+			(xy 154.94 110.49) (xy 181.61 110.49)
+		)
+		(stroke
+			(width 0)
+			(type default)
+		)
+	)
+	(wire
+		(pts
+			(xy 142.24 120.65) (xy 115.57 120.65)
+		)
+		(stroke
+			(width 0)
+			(type default)
+		)
+	)
+	(wire
+		(pts
+			(xy 157.48 46.99) (xy 160.02 46.99)
+		)
+		(stroke
+			(width 0)
+			(type default)
+		)
+	)
+	(wire
+		(pts
+			(xy 160.02 46.99) (xy 160.02 49.53)
+		)
+		(stroke
+			(width 0)
+			(type default)
+		)
+	)
+	(wire
+		(pts
+			(xy 154.94 57.15) (xy 162.56 57.15)
+		)
+		(stroke
+			(width 0)
+			(type default)
+		)
+	)
+	(wire
+		(pts
+			(xy 137.16 107.95) (xy 137.16 123.19)
+		)
+		(stroke
+			(width 0)
+			(type default)
+		)
+	)
+	(wire
+		(pts
+			(xy 113.03 128.27) (xy 142.24 128.27)
+		)
+		(stroke
+			(width 0)
+			(type default)
+		)
+	)
+	(wire
+		(pts
+			(xy 160.02 62.23) (xy 160.02 54.61)
+		)
+		(stroke
+			(width 0)
+			(type default)
+		)
+	)
+	(wire
+		(pts
+			(xy 139.7 115.57) (xy 142.24 115.57)
+		)
+		(stroke
+			(width 0)
+			(type default)
+		)
+	)
+	(wire
+		(pts
+			(xy 139.7 67.31) (xy 139.7 69.85)
+		)
+		(stroke
+			(width 0)
+			(type default)
+		)
+	)
+	(wire
+		(pts
+			(xy 154.94 113.03) (xy 184.15 113.03)
+		)
+		(stroke
+			(width 0)
+			(type default)
+		)
+	)
+	(wire
+		(pts
+			(xy 184.15 118.11) (xy 154.94 118.11)
+		)
+		(stroke
+			(width 0)
+			(type default)
+		)
+	)
+	(wire
+		(pts
+			(xy 157.48 54.61) (xy 157.48 46.99)
+		)
+		(stroke
+			(width 0)
+			(type default)
+		)
+	)
+	(wire
+		(pts
+			(xy 154.94 128.27) (xy 184.15 128.27)
+		)
+		(stroke
+			(width 0)
+			(type default)
+		)
+	)
+	(wire
+		(pts
+			(xy 134.62 64.77) (xy 142.24 64.77)
+		)
+		(stroke
+			(width 0)
+			(type default)
+		)
+	)
+	(wire
+		(pts
 			(xy 154.94 62.23) (xy 160.02 62.23)
 		)
@@
 	(wire
 		(pts
-			(xy 154.94 110.49) (xy 181.61 110.49)
-		)
-		(stroke
-			(width 0)
-			(type default)
-		)
-	)
-	(wire
-		(pts
-			(xy 142.24 120.65) (xy 115.57 120.65)
-		)
-		(stroke
-			(width 0)
-			(type default)
-		)
-	)
-	(wire
-		(pts
-			(xy 154.94 57.15) (xy 162.56 57.15)
-		)
-		(stroke
-			(width 0)
-			(type default)
-		)
-	)
-	(wire
-		(pts
-			(xy 137.16 107.95) (xy 137.16 123.19)
-		)
-		(stroke
-			(width 0)
-			(type default)
-		)
-	)
-	(wire
-		(pts
-			(xy 113.03 128.27) (xy 142.24 128.27)
-		)
-		(stroke
-			(width 0)
-			(type default)
-		)
-	)
-	(wire
-		(pts
-			(xy 139.7 115.57) (xy 142.24 115.57)
-		)
-		(stroke
-			(width 0)
-			(type default)
-		)
-	)
-	(wire
-		(pts
-			(xy 139.7 67.31) (xy 139.7 69.85)
-		)
-		(stroke
-			(width 0)
-			(type default)
-		)
-	)
-	(wire
-		(pts
-			(xy 154.94 113.03) (xy 184.15 113.03)
-		)
-		(stroke
-			(width 0)
-			(type default)
-		)
-	)
-	(wire
-		(pts
-			(xy 184.15 118.11) (xy 154.94 118.11)
-		)
-		(stroke
-			(width 0)
-			(type default)
-		)
-	)
-	(wire
-		(pts
-			(xy 154.94 128.27) (xy 184.15 128.27)
-		)
-		(stroke
-			(width 0)
-			(type default)
-		)
-	)
-	(wire
-		(pts
-			(xy 134.62 64.77) (xy 142.24 64.77)
-		)
-		(stroke
-			(width 0)
-			(type default)
-		)
-	)
-	(wire
-		(pts
 			(xy 157.48 59.69) (xy 157.48 69.85)
 		)
@@
 	(wire
 		(pts
-			(xy 160.02 62.23) (xy 160.02 54.61)
-		)
-		(stroke
-			(width 0)
-			(type default)
-		)
-	)
-	(wire
-		(pts
 			(xy 115.57 110.49) (xy 142.24 110.49)
 		)
@@
 	(wire
 		(pts
-			(xy 160.02 54.61) (xy 154.94 54.61)
-		)
-		(stroke
-			(width 0)
-			(type default)
-		)
-	)
-	(wire
-		(pts
 			(xy 181.61 120.65) (xy 154.94 120.65)
 		)
@@
 	(wire
 		(pts
+			(xy 157.48 44.45) (xy 157.48 46.99)
+		)
+		(stroke
+			(width 0)
+			(type default)
+		)
+	)
+	(wire
+		(pts
 			(xy 134.62 57.15) (xy 142.24 57.15)
 		)
@@
 		(pts
 			(xy 139.7 130.81) (xy 139.7 135.89)
-		)
-		(stroke
-			(width 0)
-			(type default)
-		)
-	)
-	(wire
-		(pts
-			(xy 160.02 52.07) (xy 160.02 54.61)
 		)
 		(stroke
@@
 		(shape output)
 		(at 162.56 64.77 0)
-		(fields_autoplaced yes)
 		(effects
 			(font
@@
 		)
 		(property "Intersheetrefs" "${INTERSHEET_REFS}"
-			(at 173.0442 64.77 0)
+			(at 181.61 39.0458 90)
 			(hide yes)
 			(show_name no)
@@
 				)
 				(justify left)
+			)
+		)
+	)
+	(symbol
+		(lib_id "Device:R_Small")
+		(at 160.02 52.07 0)
+		(unit 1)
+		(body_style 1)
+		(exclude_from_sim no)
+		(in_bom yes)
+		(on_board yes)
+		(in_pos_files yes)
+		(dnp no)
+		(fields_autoplaced yes)
+		(property "Reference" "R63"
+			(at 162.56 50.7999 0)
+			(show_name no)
+			(do_not_autoplace no)
+			(effects
+				(font
+					(size 1.016 1.016)
+				)
+				(justify left)
+			)
+		)
+		(property "Value" "10k"
+			(at 162.56 53.3399 0)
+			(show_name no)
+			(do_not_autoplace no)
+			(effects
+				(font
+					(size 1.27 1.27)
+				)
+				(justify left)
+			)
+		)
+		(property "Footprint" "Resistor_SMD:R_0603_1608Metric_Pad0.98x0.95mm_HandSolder"
+			(at 160.02 52.07 0)
+			(hide yes)
+			(show_name no)
+			(do_not_autoplace no)
+			(effects
+				(font
+					(size 1.27 1.27)
+				)
+			)
+		)
+		(property "Datasheet" ""
+			(at 160.02 52.07 0)
+			(hide yes)
+			(show_name no)
+			(do_not_autoplace no)
+			(effects
+				(font
+					(size 1.27 1.27)
+				)
+			)
+		)
+		(property "Description" "Resistor, small symbol"
+			(at 160.02 52.07 0)
+			(hide yes)
+			(show_name no)
+			(do_not_autoplace no)
+			(effects
+				(font
+					(size 1.27 1.27)
+				)
+			)
+		)
+		(pin "1"
+		)
+		(pin "2"
+		)
+		(instances
+			(project "DigiFur-Rev1.0"
+				(path "/54298b52-0ffe-40ef-8666-22993c0ca2db"
+					(reference "R63")
+					(unit 1)
+				)
 			)
 		)
@@
 	(symbol
 		(lib_id "power:+3.3V")
-		(at 160.02 52.07 0)
+		(at 157.48 44.45 0)
 		(unit 1)
 		(body_style 1)
@@
 		(fields_autoplaced yes)
 		(property "Reference" "#PWR063"
-			(at 160.02 55.88 0)
+			(at 157.48 48.26 0)
 			(hide yes)
 			(show_name no)
@@
 		)
 		(property "Value" "+3.3V_MCU"
-			(at 160.02 46.99 0)
+			(at 157.48 39.37 0)
 			(show_name no)
 			(do_not_autoplace no)
@@
 		)
 		(property "Footprint" ""
-			(at 160.02 52.07 0)
+			(at 157.48 44.45 0)
 			(hide yes)
 			(show_name no)
@@
 		)
 		(property "Datasheet" ""
-			(at 160.02 52.07 0)
+			(at 157.48 44.45 0)
 			(hide yes)
 			(show_name no)
@@
 		)
 		(property "Description" "Power symbol creates a global label with name \"+3.3V\""
-			(at 160.02 52.07 0)
-			(hide yes)
-			(show_name no)
+			(at 157.48 44.45 0)
+			(hide yes)
+			(show_name no)
