File: DigiFur-Rev1.0.kicad_pcb (KiCad board)
At the start: 4 copper layers, 158 x 80 mm, 149 parts, among them J1 705510001, J2 Micro_SD_Card_Det_Hirose_DM3AT, J3 705510001, J4 705510001, J5 Conn_02x06_Odd_Even, J6 Conn_02x09_Odd_Even, Q1 SSM3J327R, SW1 SW_Push, SW2 SW_Push, SW3 SW_Push, SW4 SW_Push, SW5 MX2A-E1NW, SW6 SW_Push, U1 TLV840MADL22DBVR, U10 USBLC6-2SC6, U11 MAX98357A, U12 TPS63900, U13 TPS63900, U14 TPS63900, U15 TPS63900, U16 TPS22917DBV, U2 NL17SZ10DBVT, U3 MCP23017x-x-SO, U4 PCF85063AT, U5 ESP32-C6-DevKitC-1, U6 TLV840MADL22DBVR, U7 TPS22917DBV, U8 OPA333 or TLV333 or TLV9041, U9 JLX256128G-931-PL_SPI, Y1 ECS-.327-12.5-34QCS-TR

Commit message: Revision to fix problems from first board fab
Parts:
- added C60: 100n, Capacitor_SMD:C_0603_1608Metric_Pad1.08x0.95mm_HandSolder, F.Cu at (120.5, 108.5)
- added C62: 10u, Capacitor_SMD:C_0603_1608Metric_Pad1.08x0.95mm_HandSolder, F.Cu at (86.2, 62.2)
- added C63: 10u, Capacitor_SMD:C_0603_1608Metric_Pad1.08x0.95mm_HandSolder, F.Cu at (89.8, 62.2)
- added C64: 10u, Capacitor_SMD:C_0603_1608Metric_Pad1.08x0.95mm_HandSolder, F.Cu at (85.8, 58.5)
- added C65: 10u, Capacitor_SMD:C_0603_1608Metric_Pad1.08x0.95mm_HandSolder, F.Cu at (92.2, 61.5)
- added JP2: SolderJumper_2_Open, Jumper:SolderJumper-2_P1.3mm_Open_TrianglePad1.0x1.5mm, F.Cu at (129.0, 110.5)
- added R46: 1M, Resistor_SMD:R_0603_1608Metric_Pad0.98x0.95mm_HandSolder, F.Cu at (124.5, 93.5)
- added R47: 0, Resistor_SMD:R_0603_1608Metric_Pad0.98x0.95mm_HandSolder, F.Cu at (74.5, 118.8)
- added R48: 0, Resistor_SMD:R_0603_1608Metric_Pad0.98x0.95mm_HandSolder, F.Cu at (74.5, 120.2)
- added R56: 0, Resistor_SMD:R_0603_1608Metric_Pad0.98x0.95mm_HandSolder, F.Cu at (127.2, 102.5)
- added R57: 0, Resistor_SMD:R_0603_1608Metric_Pad0.98x0.95mm_HandSolder, F.Cu at (91.5, 54.5)
- added R58: DNP, Resistor_SMD:R_0603_1608Metric_Pad0.98x0.95mm_HandSolder, F.Cu at (91.5, 53.0)
- added R59: 33k, Resistor_SMD:R_0603_1608Metric_Pad0.98x0.95mm_HandSolder, F.Cu at (90.8, 57.0)
- added R60: 330k, Resistor_SMD:R_0603_1608Metric_Pad0.98x0.95mm_HandSolder, F.Cu at (92.2, 57.0)
- added R61: 10k, Resistor_SMD:R_0603_1608Metric_Pad0.98x0.95mm_HandSolder, F.Cu at (88.8, 57.0)
- added R62: 330k, Resistor_SMD:R_0603_1608Metric_Pad0.98x0.95mm_HandSolder, F.Cu at (176.5, 66.0)
- added R63: 10k, Resistor_SMD:R_0603_1608Metric_Pad0.98x0.95mm_HandSolder, F.Cu at (129.8, 83.2)
- added R64: 4.7k, Resistor_SMD:R_0603_1608Metric_Pad0.98x0.95mm_HandSolder, F.Cu at (123.0, 110.8)
- added R65: 0, Resistor_SMD:R_0603_1608Metric_Pad0.98x0.95mm_HandSolder, F.Cu at (123.8, 102.5)
- added U17: SN74AXC4T774, Package_SO:TSSOP-16_4.4x5mm_P0.65mm, F.Cu at (126.0, 106.0)
- added U18: TPS2117DRL, Package_TO_SOT_SMD:SOT-583-8, F.Cu at (88.0, 60.0)
- R14, R16: value 4.7M -> 10k
- R15: value 1M -> 10k
- R25: value 300k -> 330k
- R27: value DNP -> 0
- moved R19 62.0 mm to (154.2, 58.5), turned to -90 degrees
- moved C14 62.0 mm to (159.2, 56.8)
- moved Q1 62.0 mm to (156.8, 54.8)
- moved R17 62.0 mm to (156.8, 59.2)
- moved R18 62.0 mm to (156.8, 57.8)
- moved R24 48.3 mm to (149.1, 61.5)
- moved R23 38.1 mm to (144.1, 61.5)
- moved R22 33.1 mm to (141.5, 61.5)
- moved JP1 33.0 mm to (141.5, 53.5), turned to -90 degrees
- moved C15 28.0 mm to (139.0, 61.5)
- moved C16 20.3 mm to (135.2, 60.8), turned to 0 degrees
- moved C18 20.3 mm to (135.2, 62.2), turned to 0 degrees
- moved R7 7.72 mm to (116.0, 106.0), turned to 0 degrees
- moved C1 4.51 mm to (116.5, 61.2)
- moved C2 4.51 mm to (111.8, 64.0)
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Connections:
- C11 pad 1: VBAT -> Net-(U7-VIN)
- C4 pad 1: GND -> +3.3V_MCU
- C4 pad 2: +3.3V_MCU -> GND
- C9 pad 1: VBAT -> Net-(U7-VIN)
- J1 pad 1: VBAT -> VBAT_CONN
- J2 pad 2: SPI_~{CS}_SD -> /Other Peripherals/SPI_~{CS}_SD_ISOL
- J2 pad 3: SPI_MOSI -> /Other Peripherals/SPI_MOSI_ISOL
- J2 pad 5: SPI_CLK -> /Other Peripherals/SPI_CLK_ISOL
- J2 pad 7: SPI_MISO -> /Other Peripherals/SPI_MISO_ISOL
- J5 pad 8: +3.3V_MCU -> Net-(J5-Pin_8)
- R19 pad 2: Net-(JP1-A) -> GND
- R22 pad 2: GND -> +3.3V_MCU
- R25 pad 1: SPK_EN -> Net-(R25-Pad1)
- SW1 pad 1: Net-(U3-GPB1) -> Net-(U3-GPB2)
- SW2 pad 1: Net-(U3-GPB2) -> Net-(U3-GPB3)
- SW3 pad 1: Net-(U3-GPB3) -> Net-(U3-GPB4)
- SW4 pad 1: Net-(U3-GPB4) -> Net-(U3-GPB5)
- SW5 pad 1: Net-(U3-GPB5) -> Net-(U3-GPB6)
- SW6 pad 1: Net-(U3-GPB5) -> Net-(U3-GPB6)
- U3 pad 2: Net-(U3-GPB1) -> USB_PWR
- U3 pad 7: unconnected-(U3-GPB6-Pad7) -> Net-(U3-GPB6)
- U5 pad 14: unconnected-(U5-5V0-Pad14) -> Net-(JP2-B)
- U7 pad 1: VBAT -> Net-(U7-VIN)
Routing:
- net VUSB: track 0.00 -> 126.2 mm, vias 0 -> 12
- net USB_PWR: track 0.00 -> 105.1 mm, vias 0 -> 2
- net +3.3V_MCU: track 171.4 -> 264.7 mm, vias 35 -> 29
- net Net-(U3-GPB6): track 0.00 -> 87.9 mm
- net Net-(U3-GPB1): track 84.5 -> 0.00 mm, vias 1 -> 0
- net VBAT_CONN: track 0.00 -> 73.0 mm
- net +3.3V_PERIPH: track 86.1 -> 33.7 mm, vias 27 -> 28
- net GND: track 94.4 -> 117.0 mm, vias 131 -> 164
- net Net-(J5-Pin_8): track 0.00 -> 19.4 mm
- net SPI_MISO: track 22.1 -> 5.62 mm
- net /Other Peripherals/SPI_MOSI_ISOL: track 0.00 -> 15.0 mm
- net +3.3V_SD: track 6.04 -> 20.8 mm, vias 6 -> 7
- net /Other Peripherals/SPI_MISO_ISOL: track 0.00 -> 12.1 mm
- net /Other Peripherals/SPI_~{CS}_SD_ISOL: track 0.00 -> 10.3 mm
- net LCD_D/~{C}: track 77.0 -> 66.8 mm, vias 0 -> 1
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- added copper zone on In1.Cu, net +3.3V_MCU
- added copper zone on In1.Cu, net +3.3V_PERIPH
- added copper zone on F.Cu, net Net-(JP2-B)
- added copper zone on F.Cu, net VBAT_CONN
- added copper zone on B.Cu, net VUSB
- added copper zone on F.Cu, net VUSB
- removed copper zone on B.Cu, net +3.3V_MCU
- removed copper zone on In2.Cu, net +3.3V_MCU
- removed copper zone on In2.Cu, net +3.3V_PERIPH
Other:
- board text added: "LCD Backlight"
- board text removed: "LCD Backlight:"

Commit message: Final version sent for fabrication
Parts:
- added JP3: Jumper_3_Bridged12, Connector_PinHeader_2.54mm:PinHeader_1x03_P2.54mm_Vertical, F.Cu at (90.5, 53.5)
- added R66: 1M, Resistor_SMD:R_0603_1608Metric_Pad0.98x0.95mm_HandSolder, F.Cu at (127.2, 101.0)
- R64: value 4.7k -> 3.3k
- moved R57 4.26 mm to (94.2, 57.8), turned to 180 degrees
- moved R58 4.26 mm to (94.2, 56.2), turned to 180 degrees
- moved R59 0.50 mm to (90.2, 57.0)
- moved R60 0.50 mm to (91.8, 57.0)
Routing:
- net +3.3V_MCU: track 264.7 -> 284.5 mm, vias 29 -> 30
- net Net-(U17-~{OE}): track 5.06 -> 6.56 mm
Other:
- board text added: "BAT"
- board text added: "USB"
- board text added: "USE ONLY WITH NO U18"
- board text added: "VBat Override"
